Commit message: Corrected repeated pi declaration

File: hector_quadrotor_description/urdf/quadrotor_base.urdf.xacro (robot description, xacro)
@@ -2,5 +2,5 @@
 <robot xmlns:xacro="http://www.ros.org/wiki/xacro">
   <xacro:include filename="$(find hector_sensors_description)/urdf/sonar_sensor.urdf.xacro" />
-  <xacro:property name="pi" value="3.1415926535897931" />
+  <!-- <xacro:property name="pi" value="3.1415926535897931" /> -->
   <!-- Main quadrotor link -->
   <xacro:macro name="quadrotor_base_macro">
